File: USBSerial.sch (EAGLE design)
At the start: 28 parts, among them IC1 ATMEGA16U2-MU, IC2 LD1117S33, J1 Serial, J2 ISP, J3 USB, J6 DFU, J8 Gnd, J9 VDD SELECT, Q1 16MHz

Commit message: foo
Parts:
- IC1: value ATMEGA16U2-MU -> ATMEGA16U2
- IC2: value LD1117S33 -> LD1117-33
- J1: value Serial -> ISP; device freetronics-master-v1:M06SIP -> freetronics-luke:HEADER_2X3
- J2: value ISP -> USB; device freetronics-luke:HEADER_2X3 -> freetronics-luke:USB-FT
- J3: value USB -> (none); device freetronics-luke:USB-FT -> freetronics-master-v1:M02PTH
- J4: device freetronics-master-v1:M02PTH -> freetronics-master-v1:M08STD
- J5: value (none) -> DFU; device freetronics-master-v1:M08STD -> freetronics-luke:SJ
- J6: value DFU -> Serial; device freetronics-luke:SJ -> freetronics-master-v1:M06SIP
- J9: value VDD SELECT -> VDD Select
Connections:
- net !RESET: now also J1.5; no longer J2.5
- net +3V3: no longer IC2.OUT@1
- net CTS: now also J5.2, J6.6; no longer J1.6, J6.2
- net GND: now also J1.6, J5.1; no longer J1.1, J2.6
- net MISO: now also J1.1; no longer J2.1
- net MOSI: now also J1.4; no longer J2.4
- net N$1: now also J2.GND; no longer J3.GND
- net N$115: now also J2.VBUS; no longer J3.VBUS
- net N$16: now also J2.D+; no longer J3.D+
- net N$17: now also J2.D-; no longer J3.D-
- net N$3: now also J2.SH$1, J2.SH$2, J2.SH$3, J2.SH$4; no longer J3.SH$1, J3.SH$2, J3.SH$3, J3.SH$4
- net PB0: now also J3.1; no longer J4.1
- net PB4: now also J4.8; no longer J5.8
- net PB5: now also J4.7; no longer J5.7
- net PB6: now also J4.6; no longer J5.6
- net PB7: now also J4.5; no longer J5.5
- net PC4: now also J4.1; no longer J5.1
- net PC5: now also J4.2; no longer J5.2
- net PC6: now also J4.3; no longer J5.3
- net PC7: now also J4.4; no longer J5.4
- net PD6: now also J3.2; no longer J4.2
- net RXD: now also J6.5; no longer J1.5
- net SCK: now also J1.3; no longer J2.3
- net TXD: now also J6.4; no longer J1.4
- net VDD: now also J1.2, J6.3; no longer J1.3, J2.2
Other:
- moved on the sheet: J1

Commit message: Preparation for v1.0 release
Parts:
- removed IC2: LD1117-33, freetronics-luke:LD1117-FIXED
- removed J3: (no value), freetronics-master-v1:M02PTH
- removed J4: (no value), freetronics-master-v1:M08STD
- removed J5: DFU, freetronics-luke:SJ
- removed J6: Serial, freetronics-master-v1:M06SIP
- removed J7: (no value), freetronics-master-v1:M03PTH
- removed J8: Gnd, freetronics-luke:SJ
- removed J9: VDD Select, freetronics-luke:JUMPER_SPDT
- removed L1: Ferrite bead 0805, freetronics-master-v1:INDUCTOR0805-LARGE
- removed Q1: 16MHz, freetronics-master-v1:CRYSTALHC49US
- added H1: M12PTH, freetronics-original:M12PTH
- added H2: USB-6PSMT, freetronics-jon:USB-6PSMT
- added H3: ICSP, freetronics-luke:HEADER_2X3
- added H4: Serial, freetronics-master-v1:M06SIP
- added H5: VDD Select, freetronics-luke:JUMPER_SPDT
- added L2: 0805 INDUCTOR, freetronics-master-v1:INDUCTOR0805-LARGE
- added REG1: LD1117-33 SOT-223, freetronics-luke:LD1117-FIXED
- added XTL1: 16MHz, freetronics-master-v1:CRYSTALHC49US
- added Z2: PGB1010603, freetronics:RESISTOR0603
- C1, C2: value 22p -> 22p 0603
- C3: value 100n -> 100n 0603
- C4: value 1uF -> 1uF 0603
- C5: value 10uF -> 100n 0603; device freetronics-jon:C-EUC0805 -> freetronics:CAP0603
- C6: value 100n -> 10uF 10V ceramic 0805; device freetronics:CAP0603 -> freetronics-jon:C-EUC0805
- F1: value 500mA PTC -> 500mA PTC 1812
- IC1: value ATMEGA16U2 -> ATMEGA16U2 QFN-32
- J1: value ISP -> Gnd; device freetronics-luke:HEADER_2X3 -> freetronics-jon:SJCN
- J2: value USB -> DFU; device freetronics-luke:USB-FT -> freetronics-luke:SJ
- R1: value 10k -> 10k 0603
- R2: value 1M -> 1M 0603
- R3: value 27R -> 27R 0603
- R5, R6: value 22R -> 22R 0603
- Z1: value PGB102ST23 -> PGB1010603; device freetronics-luke:PGB102ST23 -> freetronics:RESISTOR0603
Connections:
- removed net N$3: J2.SH$1, J2.SH$2, J2.SH$3, J2.SH$4, L1.1, Z1.P$3
- removed net PD6: IC1.(RTS)PD6, J3.2
- new net N$8: H2.FIX1, H2.FIX2, H2.PIN1, H2.PIN2, H2.TAB1, H2.TAB2, L2.2, Z1.2, Z2.2
- new net RTS: H4.6, IC1.(RTS)PD6
- net !RESET: now also H3.5; no longer J1.5
- net +3V3: now also C6.1, H5.1, REG1.OUT; no longer C5.1, IC2.OUT, J9.1
- net +5V: now also C5.1, H5.3, REG1.IN; no longer C6.1, IC2.IN, J9.3
- net CTS: now also H4.2, J2.2; no longer J5.2, J6.6
- net GND: now also H3.6, H4.1, J1.1, J2.1, REG1.GND; no longer IC2.GND, J1.6, J5.1, J6.1, J8.1
- net MISO: now also H3.1; no longer J1.1
- net MOSI: now also H3.4; no longer J1.4
- net N$1: now also H2.GND, J1.2, L2.1; no longer J2.GND, J8.2, L1.2
- net N$113: now also XTL1.2; no longer Q1.2
- net N$114: now also XTL1.1; no longer Q1.1
- net N$115: now also H2.VBUS; no longer J2.VBUS
- net N$16: now also H2.D+, Z1.1; no longer J2.D+, Z1.P$2
- net N$17: now also H2.D-, Z2.1; no longer J2.D-, Z1.P$1
- net PB0: now also H1.9; no longer J3.1
- net PB4: now also H1.8; no longer J4.8
- net PB5: now also H1.7; no longer J4.7
- net PB6: now also H1.6; no longer J4.6
- net PB7: now also H1.5; no longer J4.5
- net PC2: now also H1.12; no longer J7.1
- net PC4: now also H1.1; no longer J4.1
- net PC5: now also H1.2; no longer J4.2
- net PC6: now also H1.3; no longer J4.3
- net PC7: now also H1.4; no longer J4.4
- net PD0: now also H1.11; no longer J7.2
- net PD1: now also H1.10; no longer J7.3
- net RXD: now also H4.5; no longer J6.5
- net SCK: now also H3.3; no longer J1.3
- net TXD: now also H4.4; no longer J6.4
- net VDD: now also H3.2, H4.3, H5.2; no longer J1.2, J6.3, J9.2
Other:
- note added: "(C)2013 Freetronics Pty Ltd: www.freetronics.com"
- note added: "CTS (brown)"
- note added: "Freetronics USB-Serial Adapter"
- note added: "GND (black)"
- note added: "RTS (green)"
- note added: "RX (yellow)"
- note added: "TX (orange)"
- note added: "V1.0 (06-04-2013)"
- note added: "VDD (red)"
- note removed: "(C)2012 Freetronics Pty Ltd: www.freetronics.com"
- note removed: "0603"
- note removed: "0805 ceramic"
- note removed: "10V"
- note removed: "1812"
- note removed: "Freetronics ATmega16U2 breakout"
- note removed: "QFN-32"
- note removed: "SOT-223"
- note removed: "SOT-23"
- note removed: "Short on board"
- note removed: "V0.5 (06-05-2012)"
- note removed: "after DRC."
- moved on the sheet: C1, C2, C3, C4, C5, C6, F1, IC1, LED1, R1, R2, R3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
